File: Macropad_PCB/Macropad_PCB.kicad_pcb (KiCad board)
At the start: 2 copper layers, 91 x 85.5 mm, 27 parts, among them J1 OLED_128x32, SW0 RotaryEncoder, U1 MOUDLE-SEEEDUINO-XIAO

Commit message: PCB finito (in teoria)
Parts:
- U1: footprint footprints:XIAO-Generic-Hybrid-14P-2.54-21X17.8MM -> Seeed Studio XIAO Series Library:XIAO-RP2040-DIP

Commit message: Project exportation
Parts:
- D1, D10, D11, D12, D2, D3, D4, D5, D6, D7, D8, D9: footprint ScottoKeebs_Components:Diode_DO-35 -> Diode_THT:D_DO-35_SOD27_P7.62mm_Horizontal
