File: Macropad_PCB/Macropad_PCB.kicad_pcb (KiCad board)
At the start: 2 copper layers, 91 x 85.5 mm, 27 parts, among them J1 OLED_128x32, SW0 RotaryEncoder, U1 MOUDLE-SEEEDUINO-XIAO

Commit message: Update PCB
Parts:
- added REF**: MountingHole_3.2mm_M3, MountingHole:MountingHole_3.2mm_M3, F.Cu at (19.5, 33.0)
- added REF**: MountingHole_3.2mm_M3, MountingHole:MountingHole_3.2mm_M3, F.Cu at (102.5, 35.0)
- added REF**: MountingHole_3.2mm_M3, MountingHole:MountingHole_3.2mm_M3, F.Cu at (102.5, 95.0)
- U1: footprint Seeed Studio XIAO Series Library:XIAO-RP2040-DIP -> footprints:XIAO-Generic-Hybrid-14P-2.54-21X17.8MM
- moved SW0 2.50 mm to (86.7, 21.4)
- moved J1 2.48 mm to (56.1, 29.6)
Routing:
- net GND: track 50.4 -> 45.6 mm
- net +3.3V: track 33.7 -> 31.5 mm
- net SCL: track 18.2 -> 16.8 mm
- net RodeaA: track 9.57 -> 10.6 mm
- net SDA: track 8.88 -> 8.09 mm
- removed copper zone on B.Cu, net GND
- removed copper zone on F.Cu, net GND

Commit message: Added filled zone
Routing:
- added copper zone on B.Cu, net GND
- added copper zone on F.Cu, net GND
Changed lines of the file:
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@@
 		(net 26)
+	)
+	(zone
+		(net 18)
+		(net_name "GND")
+		(layers "F.Cu" "B.Cu")
+		(hatch edge 0.5)
+		(connect_pads
+			(clearance 0.5)
+		)
+		(min_thickness 0.25)
+		(filled_areas_thickness no)
+		(fill yes
+			(thermal_gap 0.5)
+			(thermal_bridge_width 0.5)
+		)
+		(polygon
+			(pts
+				(xy 11.955 11.95) (xy 110.455 12.45) (xy 110.455 102.95) (xy 11.955 102.95)
+			)
+		)
 	)
 	(embedded_fonts no)
